File: HW/aprs_test_board/aprs_test_board.kicad_pcb (KiCad board)
At the start: 2 copper layers, 48.4 x 25.5 mm, 23 parts, among them J1 Conn_Coaxial, J2 Conn_01x06, J3 Conn_01x06, U1 Si4461, Y1 30M

Commit message: pcb
Parts:
- Y1: footprint Crystal:Crystal_SMD_5032-4Pin_5.0x3.2mm -> Library:ECS3002030BDUTR
- moved Y1 0.26 mm to (98.3, 108.2)
Connections:
- Y1 pad 3: (no net) -> GND
- Y1 pad 4: (no net) -> GND
Routing:
- net Net-(J3-Pin_5): track 11.7 -> 13.3 mm
- net Net-(U1-XOUT): track 3.93 -> 5.33 mm
- net Net-(J3-Pin_6): track 13.4 -> 14.3 mm
- net GND: vias 169 -> 174
