File: HW/aprs_test_board/aprs_test_board.kicad_sch (KiCad schematic)
At the start: 19 parts, among them J1 Conn_Coaxial, J2 Conn_01x06, J3 Conn_01x06, U1 Si4461, Y1 30M

Commit message: APRS test board done
Parts:
- Y1: footprint Library:Crystal_SMD -> Crystal:Crystal_SMD_5032-4Pin_5.0x3.2mm
Connections:
- net +3.3V: now also J2.1 (Pin_1); no longer J3.1 (Pin_1)
- net GND: now also J3.1 (Pin_1); no longer J2.1 (Pin_1)
- net at J3.5 (Pin_5): now also U1.15 (~{SEL}); no longer U1.10 (GPIO1)
- net at J3.6 (Pin_6): now also U1.14 (SDI); no longer U1.9 (GPIO0)
- net at U1.11 (~{IRQ}): now also J2.4 (Pin_4); no longer J2.2 (Pin_2)
- net at J2.3 (Pin_3): now also U1.10 (GPIO1); no longer U1.12 (SCLK)
- net at U1.13 (SDO): now also J2.6 (Pin_6); no longer J2.4 (Pin_4)
- net at J2.5 (Pin_5): now also U1.12 (SCLK); no longer U1.14 (SDI)
- new net: J2.2 (Pin_2), U1.9 (GPIO0)
Other:
- moved on the sheet: J2

Commit message: test board
Parts:
- removed LX1: XX, Inductor_SMD:L_0805_2012Metric_Pad1.15x1.40mm_HandSolder, symbol Device:L
Connections:
- net at C1.2: now also C2.2, L3.1
Other:
- moved on the sheet: C2, C3, C4, C5, J1, L3, L4, L5

Commit message: pcb
Parts:
- Y1: footprint Crystal:Crystal_SMD_5032-4Pin_5.0x3.2mm -> Library:ECS3002030BDUTR
Changed lines of the file:
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@@
 			)
 		)
-		(property "Footprint" "Crystal:Crystal_SMD_5032-4Pin_5.0x3.2mm"
+		(property "Footprint" "Library:ECS3002030BDUTR"
 			(at 101.6 87.63 0)
 			(effects

Commit message: APRS testing with Arduinno
Other:
- company: (none) -> Vojtech Piroch
- title: (none) -> APRS test board
Changed lines of the file:
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@@
 	(generator_version "8.0")
 	(paper "A4")
+	(title_block
+		(title "APRS test board")
+		(date "2025-01-03")
+		(company "Vojtech Piroch")
+	)
 	(junction
 		(at 199.39 80.01)
