File: HW/picoballoon/picoballoon.kicad_pcb (KiCad board)
At the start: 4 copper layers, 55 x 63 mm, 97 parts, among them IC1 MCXC141VLH, J1 EXT_DEBUGGER, J2 Conn_01x02, U1 Si4461, U2 MPL3115A2, U4 MCP9802, U5 MAX-M10S, U6 OPA333xxDBV, Y1 30M

Commit message: little changes
Connections:
- AE1 pad 2: (no net) -> GND
- AE1 pad 3: (no net) -> GND
- AE1 pad 4: (no net) -> GND
- AE2 pad 2: (no net) -> GND
- Y1 pad 3: (no net) -> GND
- Y1 pad 4: (no net) -> GND
Changed lines of the file:
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@@
 			(size 1.25 1.6)
 			(layers "F.Cu" "F.Paste" "F.Mask")
+			(net 4 "GND")
 		)
 		(pad "4" smd rect
@@
 			(size 1.25 1.6)
 			(layers "F.Cu" "F.Paste" "F.Mask")
+			(net 4 "GND")
 		)
 		(model "${KICAD8_3DMODEL_DIR}/Crystal.3dshapes/Crystal_SMD_5032-2Pin_5.0x3.2mm.step"
@@
 			(layers "*.Cu" "*.Mask")
 			(remove_unused_layers no)
+			(net 4 "GND")
 		)
 		(model "1-5227161-7.stp"
@@
 		)
 		(model "${KICAD8_3DMODEL_DIR}/Capacitor_THT.3dshapes/C_Radial_D10.0mm_H20.0mm_P5.00mm.wrl"
+			(hide yes)
 			(offset
 				(xyz -2.5 0 0)
@@
 			(size 0.5 0.55)
 			(layers "F.Cu" "F.Paste" "F.Mask")
+			(net 4 "GND")
 		)
 		(pad "3" smd rect
@@
 			(size 0.5 1.5)
 			(layers "F.Cu" "F.Paste" "F.Mask")
+			(net 4 "GND")
 		)
 		(pad "4" smd rect
@@
 			(size 0.5 1.5)
 			(layers "F.Cu" "F.Paste" "F.Mask")
+			(net 4 "GND")
 		)
 		(model "${KIPRJMOD}/3D/RECE.20369.001E.01.stp"
