File: HW/picoballoon/picoballoon.kicad_sch (KiCad schematic)
At the start: 47 parts, among them IC1 MCXC141VLH, J1 EXT_DEBUGGER

Commit message: little changes
Parts:
- C17: value xx -> 120p
- R11: value 300 -> 470
Changed lines of the file:
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@@
 			)
 		)
-		(property "Value" "xx"
+		(property "Value" "120p"
 			(at 147.066 93.98 0)
 			(effects
@@
 			)
 		)
-		(property "Value" "300"
+		(property "Value" "470"
 			(at 96.266 34.29 0)
 			(effects

Commit message: APRS testing with Arduinno
Other:
- company: (none) -> Vojtech Piroch
- title: (none) -> MCU
Changed lines of the file:
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@@
 	(generator_version "8.0")
 	(paper "A4")
+	(title_block
+		(title "MCU")
+		(date "2025-01-03")
+		(company "Vojtech Piroch")
+	)
 	(junction
 		(at 144.78 66.04)
