File: HW/picoballoon/communication.kicad_sch (KiCad schematic)
At the start: 16 parts, among them U1 Si4461, Y1 30M

Commit message: pcb
Parts:
- C10, C16, C17, C31, C32, C33, C34, C8: footprint (none) -> Capacitor_SMD:C_0603_1608Metric_Pad1.08x0.95mm_HandSolder
- L2, L3, L6, L7, L8: footprint (none) -> Inductor_SMD:L_0603_1608Metric_Pad1.05x0.95mm_HandSolder
- Y1: footprint (none) -> Library:ECS3002030BDUTR
Changed lines of the file:
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@@
 			)
 		)
-		(property "Footprint" ""
+		(property "Footprint" "Inductor_SMD:L_0603_1608Metric_Pad1.05x0.95mm_HandSolder"
 			(at 213.36 74.93 0)
 			(effects
@@
 			)
 		)
-		(property "Footprint" ""
+		(property "Footprint" "Inductor_SMD:L_0603_1608Metric_Pad1.05x0.95mm_HandSolder"
 			(at 187.96 74.93 0)
 			(effects
@@
 			)
 		)
-		(property "Footprint" ""
+		(property "Footprint" "Inductor_SMD:L_0603_1608Metric_Pad1.05x0.95mm_HandSolder"
 			(at 175.26 74.93 0)
 			(effects
@@
 			)
 		)
-		(property "Footprint" ""
+		(property "Footprint" "Capacitor_SMD:C_0603_1608Metric_Pad1.08x0.95mm_HandSolder"
 			(at 218.7448 77.47 0)
 			(effects
@@
 			)
 		)
-		(property "Footprint" ""
+		(property "Footprint" "Capacitor_SMD:C_0603_1608Metric_Pad1.08x0.95mm_HandSolder"
 			(at 157.1752 179.07 0)
 			(effects
@@
 			)
 		)
-		(property "Footprint" ""
+		(property "Footprint" "Inductor_SMD:L_0603_1608Metric_Pad1.05x0.95mm_HandSolder"
 			(at 200.66 74.93 0)
 			(effects
@@
 			)
 		)
-		(property "Footprint" ""
+		(property "Footprint" "Library:ECS3002030BDUTR"
 			(at 124.46 82.55 0)
 			(effects
@@
 			)
 		)
-		(property "Footprint" ""
+		(property "Footprint" "Capacitor_SMD:C_0603_1608Metric_Pad1.08x0.95mm_HandSolder"
 			(at 180.6448 77.47 0)
 			(effects
@@
 			)
 		)
-		(property "Footprint" ""
+		(property "Footprint" "Capacitor_SMD:C_0603_1608Metric_Pad1.08x0.95mm_HandSolder"
 			(at 129.2352 179.07 0)
 			(effects
@@
 			)
 		)
-		(property "Footprint" ""
+		(property "Footprint" "Capacitor_SMD:C_0603_1608Metric_Pad1.08x0.95mm_HandSolder"
 			(at 143.2052 179.07 0)
 			(effects
@@
 			)
 		)
-		(property "Footprint" ""
+		(property "Footprint" "Inductor_SMD:L_0603_1608Metric_Pad1.05x0.95mm_HandSolder"
 			(at 156.21 69.85 0)
 			(effects
@@
 			)
 		)
-		(property "Footprint" ""
+		(property "Footprint" "Capacitor_SMD:C_0603_1608Metric_Pad1.08x0.95mm_HandSolder"
 			(at 168.91 73.9648 0)
 			(effects
@@
 			)
 		)
-		(property "Footprint" ""
+		(property "Footprint" "Capacitor_SMD:C_0603_1608Metric_Pad1.08x0.95mm_HandSolder"
 			(at 206.0448 77.47 0)
 			(effects
@@
 			)
 		)
-		(property "Footprint" ""
+		(property "Footprint" "Capacitor_SMD:C_0603_1608Metric_Pad1.08x0.95mm_HandSolder"
 			(at 193.3448 77.47 0)
 			(effects

Commit message: picoballoon pcb
Parts:
- AE2: footprint (none) -> Library:RECE20369001E01
Connections:
- net at C17.2, L8.1: now also C31.2; no longer L2.2
- net at L2.1: now also L7.2, U1.4 (TX); no longer C31.2
- new net: C31.1, L2.2
Other:
- moved on the sheet: C31, L2
Changed lines of the file:
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@@
 	(symbol
 		(lib_id "Device:L")
-		(at 175.26 74.93 90)
+		(at 165.1 74.93 90)
 		(unit 1)
 		(exclude_from_sim no)
@@
 		(fields_autoplaced yes)
 		(property "Reference" "L2"
-			(at 175.26 69.85 90)
+			(at 165.1 69.85 90)
 			(effects
 				(font
@@
 		)
 		(property "Value" "12n"
-			(at 175.26 72.39 90)
+			(at 165.1 72.39 90)
 			(effects
 				(font
@@
 		)
 		(property "Footprint" "Inductor_SMD:L_0603_1608Metric_Pad1.05x0.95mm_HandSolder"
-			(at 175.26 74.93 0)
+			(at 165.1 74.93 0)
 			(effects
 				(font
@@
 		)
 		(property "Datasheet" "~"
-			(at 175.26 74.93 0)
+			(at 165.1 74.93 0)
 			(effects
 				(font
@@
 		)
 		(property "Description" "Inductor"
-			(at 175.26 74.93 0)
+			(at 165.1 74.93 0)
 			(effects
 				(font
@@
 			)
 		)
-		(property "Footprint" ""
+		(property "Footprint" "Library:RECE20369001E01"
 			(at 223.52 67.31 0)
 			(effects
@@
 	(symbol
 		(lib_id "Device:C")
-		(at 165.1 74.93 90)
+		(at 175.26 74.93 90)
 		(unit 1)
 		(exclude_from_sim no)
@@
 		(fields_autoplaced yes)
 		(property "Reference" "C31"
-			(at 165.1 67.31 90)
+			(at 175.26 67.31 90)
 			(effects
 				(font
@@
 		)
 		(property "Value" "100p"
-			(at 165.1 69.85 90)
+			(at 175.26 69.85 90)
 			(effects
 				(font
@@
 		)
 		(property "Footprint" "Capacitor_SMD:C_0603_1608Metric_Pad1.08x0.95mm_HandSolder"
-			(at 168.91 73.9648 0)
+			(at 179.07 73.9648 0)
 			(effects
 				(font
@@
 		)
 		(property "Datasheet" "~"
-			(at 165.1 74.93 0)
+			(at 175.26 74.93 0)
 			(effects
 				(font
@@
 		)
 		(property "Description" "Unpolarized capacitor"
-			(at 165.1 74.93 0)
-			(effects
-				(font
+			(at 175.26 74.93 0)
+			(effects
+				(font

Commit message: test points
Parts:
- renumbered C8 to C26, C10 to C27, C16 to C28, C31 to C29, C17 to C30, C32 to C31, C33 to C32, C34 to C33, L7 to L4, L2 to L5, L8 to L6, L3 to L7, L6 to L8
Connections:
- net SDN: now reaches U1.1 (SDN)
Changed lines of the file:
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@@
+	(wire
+		(pts
+			(xy 127 74.93) (xy 133.35 74.93)
+		)
+		(stroke
+			(width 0)
+			(type default)
+		)
+	)
 	(wire
 		(pts
@@
 		)
 	)
+	(hierarchical_label "SDN"
+		(shape input)
+		(at 127 74.93 180)
+		(fields_autoplaced yes)
+		(effects
+			(font
+				(size 1.27 1.27)
+			)
+			(justify right)
+		)
+	)
 	(hierarchical_label "SO"
 		(shape input)
@@
 		(dnp no)
 		(fields_autoplaced yes)
-		(property "Reference" "L6"
+		(property "Reference" "L8"
 			(at 213.36 69.85 90)
 			(effects
@@
 			(project "picoballoon"
 				(path "/f2ac4b1c-d093-4228-80b2-7ee26b75b20f/0be041e6-a91d-4835-9904-cb6208b1f90b"
-					(reference "L6")
+					(reference "L8")
 					(unit 1)
 				)
@@
 		(dnp no)
 		(fields_autoplaced yes)
-		(property "Reference" "L8"
+		(property "Reference" "L6"
 			(at 187.96 69.85 90)
 			(effects
@@
 			(project "picoballoon"
 				(path "/f2ac4b1c-d093-4228-80b2-7ee26b75b20f/0be041e6-a91d-4835-9904-cb6208b1f90b"
-					(reference "L8")
+					(reference "L6")
 					(unit 1)
 				)
@@
 		(dnp no)
 		(fields_autoplaced yes)
-		(property "Reference" "L2"
+		(property "Reference" "L5"
 			(at 165.1 69.85 90)
 			(effects
@@
 			(project ""
 				(path "/f2ac4b1c-d093-4228-80b2-7ee26b75b20f/0be041e6-a91d-4835-9904-cb6208b1f90b"
-					(reference "L2")
+					(reference "L5")
 					(unit 1)
 				)
@@
 		(dnp no)
 		(fields_autoplaced yes)
-		(property "Reference" "C34"
+		(property "Reference" "C33"
 			(at 223.52 80.0099 0)
 			(effects
@@
 			(project "picoballoon"
 				(path "/f2ac4b1c-d093-4228-80b2-7ee26b75b20f/0be041e6-a91d-4835-9904-cb6208b1f90b"
-					(reference "C34")
+					(reference "C33")
 					(unit 1)
 				)
@@
 		(dnp no)
 		(fields_autoplaced yes)
-		(property "Reference" "C16"
+		(property "Reference" "C28"
 			(at 160.02 173.9899 0)
 			(effects
@@
 			(project "picoballoon"
 				(path "/f2ac4b1c-d093-4228-80b2-7ee26b75b20f/0be041e6-a91d-4835-9904-cb6208b1f90b"
-					(reference "C16")
+					(reference "C28")
 					(unit 1)
 				)
@@
 		(dnp no)
 		(fields_autoplaced yes)
-		(property "Reference" "L3"
+		(property "Reference" "L7"
 			(at 200.66 69.85 90)
 			(effects
@@
 			(project "picoballoon"
 				(path "/f2ac4b1c-d093-4228-80b2-7ee26b75b20f/0be041e6-a91d-4835-9904-cb6208b1f90b"
-					(reference "L3")
+					(reference "L7")
 					(unit 1)
 				)
@@
 		(dnp no)
 		(fields_autoplaced yes)
-		(property "Reference" "C17"
+		(property "Reference" "C30"
 			(at 185.42 80.0099 0)
 			(effects
@@
 			(project "picoballoon"
 				(path "/f2ac4b1c-d093-4228-80b2-7ee26b75b20f/0be041e6-a91d-4835-9904-cb6208b1f90b"
-					(reference "C17")
+					(reference "C30")
 					(unit 1)
 				)
@@
 		(dnp no)
 		(fields_autoplaced yes)
-		(property "Reference" "C8"
+		(property "Reference" "C26"
 			(at 132.08 173.9899 0)
 			(effects
@@
 			(project ""
 				(path "/f2ac4b1c-d093-4228-80b2-7ee26b75b20f/0be041e6-a91d-4835-9904-cb6208b1f90b"
-					(reference "C8")
+					(reference "C26")
 					(unit 1)
 				)
@@
 		(dnp no)
 		(fields_autoplaced yes)
-		(property "Reference" "C10"
+		(property "Reference" "C27"
 			(at 146.05 173.9899 0)
 			(effects
@@
 			(project "picoballoon"
 				(path "/f2ac4b1c-d093-4228-80b2-7ee26b75b20f/0be041e6-a91d-4835-9904-cb6208b1f90b"
-					(reference "C10")
+					(reference "C27")
 					(unit 1)
 				)
@@
 		(dnp no)
 		(fields_autoplaced yes)
-		(property "Reference" "L7"
+		(property "Reference" "L4"
 			(at 157.48 68.5799 0)
 			(effects
@@
 			(project "picoballoon"
 				(path "/f2ac4b1c-d093-4228-80b2-7ee26b75b20f/0be041e6-a91d-4835-9904-cb6208b1f90b"
-					(reference "L7")
+					(reference "L4")
 					(unit 1)
 				)
@@
 		(dnp no)
 		(fields_autoplaced yes)
-		(property "Reference" "C31"
+		(property "Reference" "C29"
 			(at 175.26 67.31 90)
 			(effects
@@
 			(project ""
 				(path "/f2ac4b1c-d093-4228-80b2-7ee26b75b20f/0be041e6-a91d-4835-9904-cb6208b1f90b"
-					(reference "C31")
+					(reference "C29")
 					(unit 1)
 				)
@@
 		(dnp no)
 		(fields_autoplaced yes)
-		(property "Reference" "C33"
+		(property "Reference" "C32"
 			(at 210.82 80.0099 0)
 			(effects
@@
 			(project "picoballoon"
 				(path "/f2ac4b1c-d093-4228-80b2-7ee26b75b20f/0be041e6-a91d-4835-9904-cb6208b1f90b"
-					(reference "C33")
+					(reference "C32")
 					(unit 1)
 				)
@@
 		(dnp no)
 		(fields_autoplaced yes)
-		(property "Reference" "C32"
+		(property "Reference" "C31"
 			(at 198.12 80.0099 0)
 			(effects
@@
 			(project "picoballoon"
 				(path "/f2ac4b1c-d093-4228-80b2-7ee26b75b20f/0be041e6-a91d-4835-9904-cb6208b1f90b"
-					(reference "C32")
-					(unit 1)
-				)
+					(reference "C31")
+					(unit 1)
+				)

Commit message: mcxc
Parts:
- AE2: footprint Library:RECE20369001E01 -> Library:BNC_Connector_PCB
Changed lines of the file:
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@@
 			)
 		)
-		(property "Footprint" "Library:RECE20369001E01"
+		(property "Footprint" "Library:BNC_Connector_PCB"
 			(at 223.52 67.31 0)
 			(effects

Commit message: APRS testing with Arduinno
Other:
- company: (none) -> Vojtech Piroch
- title: (none) -> Communication
Changed lines of the file:
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@@
 	(generator_version "8.0")
 	(paper "A4")
+	(title_block
+		(title "Communication")
+		(date "2025-01-03")
+		(company "Vojtech Piroch")
+	)
 	(junction
 		(at 194.31 87.63)

Commit message: bom
Parts:
- C30: value 14,35p -> 15p
- C32: value 43,06p -> 43p
- L4: value 552n -> 480n
- L6: value 106n -> 110n
- L7, L8: value 74,74n -> 75n
Changed lines of the file:
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@@
 			)
 		)
-		(property "Value" "74,74n"
+		(property "Value" "75n"
 			(at 213.36 72.39 90)
 			(effects
@@
 			)
 		)
-		(property "Value" "106n"
+		(property "Value" "110n"
 			(at 187.96 72.39 90)
 			(effects
@@
 			)
 		)
-		(property "Value" "74,74n"
+		(property "Value" "75n"
 			(at 200.66 72.39 90)
 			(effects
@@
 			)
 		)
-		(property "Value" "14,35p"
+		(property "Value" "15p"
 			(at 185.42 82.5499 0)
 			(effects
@@
 			)
 		)
-		(property "Value" "552n"
+		(property "Value" "480n"
 			(at 157.48 71.1199 0)
 			(effects
@@
 			)
 		)
-		(property "Value" "43,06p"
+		(property "Value" "43p"
 			(at 210.82 82.5499 0)
 			(effects
