File: HW/picoballoon_v2/picoballoon.kicad_sch (KiCad schematic)
At the start: 37 parts, among them IC1 MCXC141VLH, J1 EXT_DEBUGGER

Commit message: little changes in scheme
Other:
- sheet GNSS ports: added EN; removed none
- moved on the sheet: R3, R4

Commit message: PCB v2
Parts:
- removed R10, R9: 10k, Resistor_SMD:R_0603_1608Metric_Pad0.98x0.95mm_HandSolder, symbol Device:R
Connections:
- net GNSS_EN: now also IC1.61 (PTD4/LLWU_P14)
- net GNSS_RESET: now also IC1.60 (PTD3); no longer IC1.61 (PTD4/LLWU_P14)
- net at C17.1, R14.2: now also IC1.18 (PTE30); no longer IC1.9 (PTE20)
- net SCL_TEMP: no longer names the net of IC1.37 (PTB2)
- net SDA_TEMP: no longer names the net of IC1.38 (PTB3)
Other:
- sheet sensors ports: added none; removed SCL_TEMP, SDA_TEMP
- moved on the sheet: C16, C17, C37, J1, R12, R13, R14, R15, R16, R2, R5, R6
