File: HW/picoballoon_v2/sensors.kicad_sch (KiCad schematic)
At the start: 8 parts, among them U2 MPL3115A2, U4 MCP9802

Commit message: PCB v2
Connections:
- net SCL_TEMP is gone; now on net SCL: U4.4 (SCLK)
- net SDA_TEMP is gone; now on net SDA: U4.5 (SDA)
Changed lines of the file:
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@@
 	(wire
 		(pts
-			(xy 40.64 49.53) (xy 50.8 49.53)
-		)
-		(stroke
-			(width 0)
-			(type default)
-		)
-	)
-	(wire
-		(pts
-			(xy 40.64 52.07) (xy 50.8 52.07)
+			(xy 44.45 49.53) (xy 50.8 49.53)
+		)
+		(stroke
+			(width 0)
+			(type default)
+		)
+	)
+	(wire
+		(pts
+			(xy 44.45 52.07) (xy 50.8 52.07)
 		)
 		(stroke
@@
 	(wire
 		(pts
-			(xy 151.13 175.26) (xy 161.29 175.26)
-		)
-		(stroke
-			(width 0)
-			(type default)
-		)
-	)
-	(wire
-		(pts
 			(xy 228.6 59.69) (xy 228.6 60.96)
 		)
@@
 		(pts
 			(xy 205.74 41.91) (xy 205.74 39.37)
-		)
-		(stroke
-			(width 0)
-			(type default)
-		)
-	)
-	(wire
-		(pts
-			(xy 151.13 177.8) (xy 161.29 177.8)
 		)
 		(stroke
@@
 		)
 	)
-	(label "SDA_TEMP"
-		(at 40.64 49.53 0)
-		(fields_autoplaced yes)
-		(effects
-			(font
-				(size 1.27 1.27)
-			)
-			(justify left bottom)
-		)
-	)
-	(label "SDA_TEMP"
-		(at 151.13 175.26 0)
-		(fields_autoplaced yes)
-		(effects
-			(font
-				(size 1.27 1.27)
-			)
-			(justify left bottom)
-		)
-	)
-	(label "SCL_TEMP"
-		(at 151.13 177.8 0)
-		(fields_autoplaced yes)
-		(effects
-			(font
-				(size 1.27 1.27)
-			)
-			(justify left bottom)
-		)
-	)
-	(label "SCL_TEMP"
-		(at 40.64 52.07 0)
+	(label "SDA"
+		(at 44.45 49.53 0)
+		(fields_autoplaced yes)
+		(effects
+			(font
+				(size 1.27 1.27)
+			)
+			(justify left bottom)
+		)
+	)
+	(label "SCL"
+		(at 44.45 52.07 0)
 		(fields_autoplaced yes)
 		(effects
@@
 			)
 			(justify right bottom)
-		)
-	)
-	(hierarchical_label "SDA_TEMP"
-		(shape bidirectional)
-		(at 161.29 175.26 0)
-		(fields_autoplaced yes)
-		(effects
-			(font
-				(size 1.27 1.27)
-			)
-			(justify left)
 		)
 	)
@@
 		(fields_autoplaced yes)
 		(effects
-			(font
-				(size 1.27 1.27)
-			)
-			(justify left)
-		)
-	)
-	(hierarchical_label "SCL_TEMP"
-		(shape input)
-		(at 161.29 177.8 0)
-		(fields_autoplaced yes)
-		(effects
