File: HW/picoballoon_v2/GNSS.kicad_sch (KiCad schematic)
At the start: 4 parts, among them J3 Conn_Coaxial, U5 MAX-M10S

Commit message: little changes in scheme
Parts:
- added Q1: PMOS, symbol Simulation_SPICE:PMOS
- added R19: 10k, symbol Device:R
- added R20: R, symbol Device:R
- added R21: 0, symbol Device:R
Connections:
- net +3.3V: now also Q1.3 (S), R19.1, R21.1; no longer U5.6 (V_BCKP), U5.7 (VCC_IO), U5.8 (VCC)
- new net: Q1.1 (D), R21.2, U5.6 (V_BCKP), U5.7 (VCC_IO), U5.8 (VCC)
- new net: Q1.2 (G), R19.2, R20.2
- new net EN: R20.1

Commit message: PCB v2
Parts:
- removed C25: 100n, Capacitor_SMD:C_0603_1608Metric_Pad1.08x0.95mm_HandSolder, symbol Device:C
- J3: footprint (none) -> Connector_Coaxial:U.FL_Molex_MCRF_73412-0110_Vertical
- Q1: footprint (none) -> Library:SOT95P237X112-3N
- R19, R21: footprint (none) -> Resistor_SMD:R_0603_1608Metric_Pad0.98x0.95mm_HandSolder
- R20: value R -> 875; footprint (none) -> Resistor_SMD:R_0603_1608Metric_Pad0.98x0.95mm_HandSolder
Connections:
- net +3.3V: no longer C24.1
- net at Q1.1 (D), R21.2, U5.6 (V_BCKP)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: now also C24.1
Other:
- moved on the sheet: C24, J3, R21

Commit message: pcb v2
Parts:
- R21: now not fitted
Changed lines of the file:
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@@
 		(in_bom yes)
 		(on_board yes)
-		(dnp no)
+		(dnp yes)
 		(property "Reference" "R21"
 			(at 120.396 69.85 0)
